File: Woggle/Woggle.kicad_pcb (KiCad board)
At the start: 2 copper layers, 18 parts, among them J1 ICSP, U1 ATtiny85-20P

Commit message: .
Parts:
- added Lanyard1: MountingHole, MountingHole:MountingHole_5mm, F.Cu at (75.7, 58.0)
- D1: value 2a -> 1a
- D10: value 4b -> 5b
- D2: value 2b -> 2a
- D4: value 3b -> 1b
- D5: value 5a -> 2b
- D6: value 5b -> 3b
- D7: value 1a -> 4a
- D8: value 1b -> 4b
- D9: value 4a -> 5a
- moved D12 118.2 mm to (74.4, 146.3)
- moved D9 114.7 mm to (65.3, 137.7)
- moved D5 103.7 mm to (56.1, 102.1)
- moved D10 94.1 mm to (89.2, 137.7), turned to 180 degrees
- moved D7 91.4 mm to (58.2, 120.4)
- moved D3 80.4 mm to (58.2, 85.3)
- moved D11 77.7 mm to (77.0, 67.1)
- moved D8 67.1 mm to (95.8, 120.4), turned to 180 degrees
- moved D6 64.2 mm to (98.3, 102.1), turned to 180 degrees
- moved D1 59.7 mm to (65.3, 67.1)
- moved J1 57.9 mm to (62.7, 74.7)
- moved R2 55.5 mm to (75.2, 76.7), turned to 180 degrees
- moved R1 52.8 mm to (75.2, 79.8), turned to 180 degrees
- moved R4 48.6 mm to (88.4, 76.7), turned to 0 degrees
- moved R3 46.1 mm to (88.4, 79.8), turned to 0 degrees
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Connections:
- D10 pad 1: Net-(D10-K) -> Net-(D1-K)
- D10 pad 2: Net-(D1-K) -> Net-(D10-A)
- D11 pad 1: Net-(D11-K) -> Net-(D10-A)
- D11 pad 2: Net-(D10-K) -> Net-(D1-A)
- D12 pad 1: Net-(D10-K) -> Net-(D1-A)
- D12 pad 2: Net-(D11-K) -> Net-(D10-A)
- D2 pad 1: Net-(D1-A) -> Net-(D2-K)
- D3 pad 1: Net-(D11-K) -> Net-(D10-A)
- D3 pad 2: Net-(D1-K) -> Net-(D2-K)
- D4 pad 1: Net-(D1-K) -> Net-(D1-A)
- D4 pad 2: Net-(D11-K) -> Net-(D1-K)
- D5 pad 1: Net-(D11-K) -> Net-(D1-K)
- D5 pad 2: Net-(D1-A) -> Net-(D2-K)
- D6 pad 1: Net-(D1-A) -> Net-(D2-K)
- D6 pad 2: Net-(D11-K) -> Net-(D10-A)
- D7 pad 1: Net-(D1-A) -> Net-(D2-K)
- D7 pad 2: Net-(D10-K) -> Net-(D1-A)
- D8 pad 1: Net-(D10-K) -> Net-(D1-A)
- D8 pad 2: Net-(D1-A) -> Net-(D2-K)
- D9 pad 1: Net-(D1-K) -> Net-(D10-A)
- D9 pad 2: Net-(D10-K) -> Net-(D1-K)
- R1 pad 2: Net-(D10-K) -> Net-(D1-A)
- R2 pad 2: Net-(D1-A) -> Net-(D1-K)
- R3 pad 2: Net-(D1-K) -> Net-(D2-K)
- R4 pad 2: Net-(D11-K) -> Net-(D10-A)
Routing:
- net Net-(D2-K): track 0.00 -> 214.0 mm, vias 0 -> 4
- net Net-(D10-A): track 0.00 -> 173.7 mm, vias 0 -> 2
- net Net-(D1-K): track 62.6 -> 198.5 mm
- net Net-(D1-A): track 87.6 -> 203.9 mm, vias 0 -> 2
- net Net-(D10-K): track 74.9 -> 0.00 mm
- net Net-(D11-K): track 62.6 -> 0.00 mm
- net /SCK/ARD13: track 16.5 -> 34.3 mm
- net /Reset/ARD10: track 9.30 -> 26.5 mm
- net /MOSI/ARD11: track 14.3 -> 30.4 mm, vias 0 -> 1
- net GND: track 14.8 -> 30.3 mm, vias 0 -> 1
- net +VE: track 5.61 -> 17.5 mm
- net Net-(U1-XTAL1/PB3): track 12.1 -> 2.90 mm
- net Net-(U1-XTAL2/PB4): track 12.1 -> 2.90 mm
- net /MISO/ARD12: track 16.2 -> 17.4 mm
Other:
- board outline added: 49 x 99 mm

Commit message: .
Parts:
- removed J1: ICSP, Connector_PinHeader_2.54mm:PinHeader_2x03_P2.54mm_Vertical
- added SW1: SW_SPDT, Button_Switch_THT:SW_Slide_SPDT_Angled_CK_OS102011MA1Q, F.Cu at (59.1, 74.2)
- added SW2: SW_Push, Button_Switch_THT:SW_PUSH-12mm, F.Cu at (81.8, 77.4)
- R1, R2, R3, R4: value R_Small -> 390
- moved R2 16.1 mm to (68.6, 91.4)
- moved R4 13.5 mm to (82.5, 88.9)
- moved U1 13.5 mm to (79.4, 94.0)
- moved R3 13.1 mm to (82.5, 91.4)
- moved R1 11.3 mm to (68.6, 88.9)
- moved D11 9.27 mm to (76.8, 57.8)
- moved Lanyard1 7.83 mm to (83.2, 60.3)
- moved D12 2.45 mm to (76.8, 146.7), turned to 180 degrees
Connections:
- R1 pad 1: /SCK/ARD13 -> /MISO/ARD12
- R2 pad 1: /MISO/ARD12 -> /SCK/ARD13
Routing:
- net +VE: track 17.5 -> 51.3 mm, vias 0 -> 1
- net /SCK/ARD13: track 34.3 -> 3.17 mm
- net GND: track 30.3 -> 0.00 mm, vias 1 -> 0
- net Net-(D1-A): track 203.9 -> 231.6 mm
- net Net-(D10-A): track 173.7 -> 201.2 mm, vias 2 -> 3
- net /Reset/ARD10: track 26.5 -> 0.00 mm
- net /MISO/ARD12: track 17.4 -> 3.17 mm
- net Net-(D2-K): track 214.0 -> 226.5 mm
- net Net-(D1-K): track 198.5 -> 210.8 mm, vias 0 -> 2
- net /MOSI/ARD11: track 30.4 -> 21.7 mm, vias 1 -> 0

Commit message: .
Parts:
- added J1: ICSP, Connector:Tag-Connect_TC2030-IDC-NL_2x03_P1.27mm_Vertical, F.Cu at (87.6, 77.5)
Routing:
- net /Reset/ARD10: track 0.00 -> 25.1 mm, vias 0 -> 2
- net /SCK/ARD13: track 3.17 -> 25.4 mm, vias 0 -> 2
- net /MISO/ARD12: track 3.17 -> 25.2 mm, vias 0 -> 2
- net /MOSI/ARD11: track 21.7 -> 42.6 mm
- net +VE: track 51.3 -> 70.3 mm
- net GND: track 0.00 -> 13.5 mm, vias 0 -> 2

Commit message: .
Parts:
- added D13: Blink, LED_THT:LED_D5.0mm, F.Cu at (64.8, 100.3)
- added D14: Power, LED_THT:LED_D5.0mm, F.Cu at (88.9, 100.3)
- added D15: BZT52, Diode_THT:D_5W_P10.16mm_Horizontal, F.Cu at (80.6, 115.6)
- added D16: 1N4148, Diode_THT:D_5W_P10.16mm_Horizontal, F.Cu at (80.6, 109.9)
- added D17: BZT52, Diode_THT:D_5W_P10.16mm_Horizontal, F.Cu at (80.6, 120.4)
- added R5: 1K, Resistor_THT:R_Axial_DIN0207_L6.3mm_D2.5mm_P10.16mm_Horizontal, F.Cu at (82.5, 95.2)
- added R6: 1K5, Resistor_THT:R_Axial_DIN0207_L6.3mm_D2.5mm_P10.16mm_Horizontal, F.Cu at (80.6, 105.4)
- added R7: 68R, Resistor_THT:R_Axial_DIN0207_L6.3mm_D2.5mm_P10.16mm_Horizontal, F.Cu at (70.5, 97.8)
- added R8: 68R, Resistor_THT:R_Axial_DIN0207_L6.3mm_D2.5mm_P10.16mm_Horizontal, F.Cu at (70.5, 101.6)
- added R9: 1K, Resistor_THT:R_Axial_DIN0207_L6.3mm_D2.5mm_P10.16mm_Horizontal, F.Cu at (68.6, 95.2)
- added REF**: KiCad-Logo2_5mm_SilkScreen, Symbol:KiCad-Logo2_5mm_SilkScreen, B.Cu at (75.6, 141.0)
- added SW3: Reset, Button_Switch_THT:SW_PUSH-12mm, F.Cu at (69.3, 129.6)
- added X1: USB-A-H, Connector_USB:USB_B_Lumberg_2411_02_Horizontal, F.Cu at (84.7, 109.9)
- R1, R2, R3, R4: footprint Resistor_THT:R_Axial_DIN0204_L3.6mm_D1.6mm_P5.08mm_Horizontal -> Resistor_THT:R_Axial_DIN0207_L6.3mm_D2.5mm_P10.16mm_Horizontal
- SW2: value SW_Push -> Sequance
- moved R2 0.64 mm to (68.6, 92.1)
- moved R3 0.64 mm to (82.5, 92.1)
Routing:
- net GND: track 13.5 -> 137.5 mm, vias 2 -> 3
- net /Reset/ARD10: track 25.1 -> 77.1 mm, vias 2 -> 1
- net /D+: track 0.00 -> 45.3 mm
- net /D-: track 0.00 -> 41.7 mm
- net Net-(U1-XTAL2/PB4): track 3.18 -> 20.9 mm
- net Net-(D16-A): track 0.00 -> 16.7 mm
- net +5V: track 0.00 -> 14.5 mm
- net Net-(D13-K): track 0.00 -> 10.3 mm
- net Net-(U1-XTAL1/PB3): track 3.18 -> 11.4 mm
- net Net-(D10-A): track 201.2 -> 208.1 mm
- net Net-(D14-K): track 0.00 -> 6.66 mm
- net Net-(D1-K): track 210.8 -> 204.6 mm, vias 2 -> 1
- net Net-(D2-K): track 226.5 -> 220.7 mm, vias 4 -> 3
- net /MOSI/ARD11: track 42.6 -> 40.7 mm, vias 0 -> 1
- net +VE: track 70.3 -> 71.4 mm
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