File: Woggle/Woggle.kicad_pcb (KiCad board)
At the start: 2 copper layers, 49 x 99 mm, 34 parts, among them J1 ICSP, SW1 SW_SPDT, SW2 Sequance, SW3 Reset, U1 ATtiny85-20P, X1 USB-A-H

Commit message: .
Parts:
- removed X1: USB-A-H, Connector_USB:USB_B_Lumberg_2411_02_Horizontal
- added J2: USB_Program, Connector_PinHeader_2.54mm:PinHeader_1x04_P2.54mm_Vertical, F.Cu at (95.0, 107.7)
- Lanyard1: value MountingHole -> Lanyard
Routing:
- net Net-(D16-A): track 16.7 -> 27.9 mm, vias 0 -> 1
- net /D-: track 41.7 -> 52.2 mm, vias 0 -> 1
- net /D+: track 45.3 -> 53.8 mm, vias 0 -> 1
- net GND: track 137.5 -> 130.3 mm
- net Net-(D1-K): track 204.6 -> 205.3 mm, vias 1 -> 2
- net Net-(U1-XTAL2/PB4): track 20.9 -> 20.6 mm, vias 0 -> 1
- net Net-(D1-A): vias 2 -> 4
- net Net-(D2-K): vias 3 -> 4
- net Net-(D10-A): vias 3 -> 4

Commit message: .
Parts:
- added REF**: Not Prefered, Connector_PinSocket_2.54mm:PinSocket_1x03_P2.54mm_Vertical, F.Cu at (141.6, 93.4)
- added REF**: Not Prefered, Connector_PinSocket_2.54mm:PinSocket_1x03_P2.54mm_Vertical, F.Cu at (141.7, 69.1)
- added REF**: Prefered, Connector_PinSocket_2.54mm:PinSocket_1x03_P2.54mm_Vertical, F.Cu at (131.5, 69.2)
Routing:
- net (no net): track 0.00 -> 19.8 mm

Commit message: .
Parts:
- removed D13: Blink, LED_THT:LED_D5.0mm
- removed D14: Power, LED_THT:LED_D5.0mm
- removed D15, D17: BZT52, Diode_THT:D_5W_P10.16mm_Horizontal
- removed D16: 1N4148, Diode_THT:D_5W_P10.16mm_Horizontal
- removed J1: ICSP, Connector:Tag-Connect_TC2030-IDC-NL_2x03_P1.27mm_Vertical
- removed J2: USB_Program, Connector_PinHeader_2.54mm:PinHeader_1x04_P2.54mm_Vertical
- removed R5, R9: 1K, Resistor_THT:R_Axial_DIN0207_L6.3mm_D2.5mm_P10.16mm_Horizontal
- removed R6: 1K5, Resistor_THT:R_Axial_DIN0207_L6.3mm_D2.5mm_P10.16mm_Horizontal
- removed R7, R8: 68R, Resistor_THT:R_Axial_DIN0207_L6.3mm_D2.5mm_P10.16mm_Horizontal
- removed the REF** at (141.6, 93.4)
- removed the REF** at (141.7, 69.1)
- removed the REF** at (131.5, 69.2)
- removed SW3: Reset, Button_Switch_THT:SW_PUSH-12mm
- added BT1: 2 x AAA, Scouts:2 x AAA battery cell holder, B.Cu at (69.2, 86.0)
- D1, D10, D11, D12, D2, D3, D4, D5, D6, D7, D8, D9: footprint LED_THT:LED_D5.0mm -> Scouts:5mm LED
- U1: footprint Package_DIP:DIP-8_W7.62mm -> Scouts:DIP 8
- moved U1 3.18 mm to (79.4, 97.2)
- moved R1 2.54 mm to (68.6, 91.4)
- moved R2 2.54 mm to (68.6, 94.6)
- moved R3 2.54 mm to (82.5, 94.6)
- moved R4 2.54 mm to (82.5, 91.4)
Connections:
- net /MISO/ARD12 renamed Net-(U1-PB1)
- net /MOSI/ARD11 renamed Net-(U1-AREF/PB0)
- net /SCK/ARD13 renamed Net-(U1-PB2)
- U1 pad 1: /Reset/ARD10 -> unconnected-(U1-~{RESET}/PB5-Pad1)
Routing:
- net GND: track 130.3 -> 6.12 mm, vias 3 -> 1
- net /Reset/ARD10: track 77.1 -> 0.00 mm, vias 1 -> 0
- net /D+: track 53.8 -> 0.00 mm, vias 1 -> 0
- net /D-: track 52.2 -> 0.00 mm, vias 1 -> 0
- net Net-(D2-K): track 220.7 -> 169.3 mm, vias 4 -> 5
- net Net-(D1-K): track 205.3 -> 170.2 mm, vias 2 -> 6
- net Net-(D10-A): track 208.1 -> 179.8 mm, vias 4 -> 5
- net Net-(D16-A): track 27.9 -> 0.00 mm, vias 1 -> 0
- net Net-(D1-A): track 231.7 -> 207.2 mm, vias 4 -> 7
- net Net-(U1-PB2): track 25.7 -> 3.17 mm
- net Net-(U1-PB1): track 25.2 -> 3.44 mm
- net (no net): track 19.8 -> 0.00 mm
- net Net-(U1-XTAL2/PB4): track 20.6 -> 3.44 mm, vias 1 -> 0
- net Net-(BT1-+): track 0.00 -> 15.6 mm, vias 0 -> 1
- net Net-(U1-AREF/PB0): track 40.7 -> 25.1 mm, vias 1 -> 0
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
Commit message: .
Parts:
- D1: value 1a -> 1
- D10: value 5b -> 7
- D11: value 6a -> 2
- D12: value 6b -> 3
- D2: value 2a -> 10
- D3: value 3a -> 5
- D4: value 1b -> 0
- D5: value 2b -> 11
- D6: value 3b -> 4
- D7: value 4a -> 8
- D8: value 4b -> 9
- D9: value 5a -> 6
- moved D3 59.9 mm to (88.3, 137.2), turned to 0 degrees
- moved D12 48.4 mm to (95.9, 102.2), turned to 0 degrees
- moved D8 46.2 mm to (53.3, 102.2), turned to 0 degrees
- moved D2 39.3 mm to (54.6, 85.7), turned to 0 degrees
- moved D4 36.5 mm to (74.3, 55.9), turned to 0 degrees
- moved D5 35.1 mm to (61.0, 67.3), turned to 0 degrees
- moved D11 32.8 mm to (94.0, 85.7), turned to 0 degrees
- moved D10 28.2 mm to (61.0, 137.2), turned to 0 degrees
- moved D1 23.0 mm to (88.3, 67.3), turned to 0 degrees
- moved D6 19.0 mm to (94.0, 120.7), turned to 0 degrees
- moved D9 14.2 mm to (74.3, 148.6), turned to 0 degrees
- moved R3 10.2 mm to (92.7, 95.2), turned to 180 degrees
- moved R4 10.2 mm to (92.7, 90.8), turned to 180 degrees
- moved D7 2.94 mm to (55.2, 120.7), turned to 0 degrees
- moved R2 0.64 mm to (68.6, 95.2)
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Connections:
- R3 pad 1: Net-(U1-XTAL1/PB3) -> Net-(D2-K)
- R3 pad 2: Net-(D2-K) -> Net-(U1-XTAL1/PB3)
- R4 pad 1: Net-(U1-XTAL2/PB4) -> Net-(D10-A)
- R4 pad 2: Net-(D10-A) -> Net-(U1-XTAL2/PB4)
Routing:
- net Net-(D10-A): track 179.8 -> 116.2 mm, vias 5 -> 2
- net Net-(D1-A): track 207.2 -> 151.6 mm
- net Net-(D1-K): track 170.2 -> 154.0 mm, vias 6 -> 4
- net Net-(D2-K): track 169.3 -> 157.3 mm, vias 5 -> 7
- net +VE: track 59.7 -> 57.1 mm
- net Net-(BT1-+): track 15.6 -> 16.3 mm
- net Net-(U1-XTAL2/PB4): track 3.44 -> 4.07 mm
- net Net-(U1-PB1): track 3.44 -> 4.07 mm
- net Net-(U1-AREF/PB0): track 25.1 -> 25.4 mm, vias 0 -> 2
Other:
- board text added: "https://wokwi.com/projects/454604516673417217"

Commit message: .
Parts:
- added G***: LOGO, Scouts:1st Byfield, F.Cu at (75.6, 115.6)
- moved R3 34.6 mm to (58.4, 90.8), turned to 0 degrees
- moved R4 34.6 mm to (58.4, 95.2), turned to 0 degrees
- moved R1 14.7 mm to (82.5, 95.2), turned to 0 degrees
- moved R2 14.7 mm to (82.5, 90.8), turned to 0 degrees
- moved U1 10.8 mm to (71.8, 89.5), turned to 0 degrees
- moved D11 0.64 mm to (94.6, 85.7)
- moved Lanyard1 0.63 mm to (83.2, 61.0)
- moved SW1 0.09 mm to (59.1, 74.2)
Routing:
- net Net-(D1-K): track 154.0 -> 187.9 mm
- net Net-(D10-A): track 116.2 -> 150.0 mm, vias 2 -> 3
- net GND: track 5.75 -> 18.1 mm
- net Net-(U1-AREF/PB0): track 25.4 -> 36.2 mm
- net +VE: track 57.1 -> 48.0 mm, vias 0 -> 2
- net Net-(D2-K): track 157.3 -> 154.2 mm, vias 7 -> 8
- net Net-(D1-A): track 151.6 -> 152.7 mm, vias 7 -> 6
- net Net-(U1-XTAL2/PB4): track 4.07 -> 3.44 mm
- net Net-(U1-PB1): track 4.07 -> 3.44 mm

Commit message: .
Parts:
- added C1: 10pF, Capacitor_THT:C_Disc_D4.7mm_W2.5mm_P5.00mm, F.Cu at (85.8, 74.3)
- added C2: 100nF, Capacitor_THT:C_Disc_D4.7mm_W2.5mm_P5.00mm, F.Cu at (85.8, 79.4)
- D1: value 1 -> LED 1
- D10: value 7 -> LED 7
- D11: value 2 -> LED 2
- D12: value 3 -> LED 3
- D2: value 10 -> LED 10
- D3: value 5 -> LED 5
- D4: value 0 -> LED 0
- D5: value 11 -> LED 11
- D6: value 4 -> LED 4
- D7: value 8 -> LED 8
- D8: value 9 -> LED 9
- D9: value 6 -> LED 6
- moved R1 1.91 mm to (84.5, 95.2)
- moved R2 1.91 mm to (84.5, 90.8)
- moved R3 1.91 mm to (56.5, 90.8)
- moved R4 1.91 mm to (56.5, 95.2)
Routing:
- net GND: track 18.1 -> 43.9 mm, vias 1 -> 2
- net +VE: track 48.0 -> 69.5 mm, vias 2 -> 4
- net Net-(D10-A): track 150.0 -> 154.6 mm
- net Net-(D1-A): track 152.7 -> 157.2 mm
- net Net-(D1-K): track 187.9 -> 192.3 mm
- net Net-(D2-K): track 154.2 -> 151.5 mm
- net Net-(U1-PB1): track 3.44 -> 5.34 mm
- net Net-(U1-XTAL2/PB4): track 3.44 -> 5.34 mm
- net Net-(U1-XTAL1/PB3): track 3.70 -> 5.61 mm
- net Net-(U1-PB2): track 3.70 -> 5.61 mm

Commit message: .
Parts:
- BT1: footprint Scouts:2 x AAA battery cell holder -> Scouts:Scouts - 2 x AAA battery cell holder
- D1, D10, D11, D12, D2, D3, D4, D5, D6, D7, D8, D9: footprint Scouts:5mm LED -> Scouts:Scouts - 5mm LED
- R1, R2, R3, R4: footprint Resistor_THT:R_Axial_DIN0207_L6.3mm_D2.5mm_P10.16mm_Horizontal -> Scouts:Scouts - Resistor (10.16mm)
- U1: footprint Scouts:DIP 8 -> Scouts:Scouts - DIP 8
- moved R1 0.64 mm to (84.5, 95.9)
- moved R4 0.64 mm to (56.5, 95.9)
Routing:
- net Net-(D1-K): track 192.3 -> 194.0 mm
- net Net-(D2-K): track 151.5 -> 150.6 mm
