File: Woggle/Woggle.kicad_pcb (KiCad board)
At the start: 2 copper layers, 49 x 99 mm, 25 parts, among them SW1 SW_SPDT, SW2 Sequance, U1 ATtiny85-20P

Commit message: .
Parts:
- added REF**: SquashedFlySilk, KiCad Footprints:SquashedFlySilk, B.Cu at (75.6, 63.5)
- moved BT1 0.23 mm to (69.2, 85.7)
Routing:
- net Net-(D1-A): track 157.4 -> 162.8 mm
- net +VE: track 69.5 -> 65.9 mm, vias 4 -> 2
- net Net-(D2-K): track 150.6 -> 148.2 mm
- net GND: track 43.9 -> 45.6 mm
- net Net-(U1-AREF/PB0): track 36.2 -> 34.8 mm
- net Net-(D1-K): track 194.0 -> 193.4 mm
- net Net-(D10-A): track 154.3 -> 153.9 mm, vias 3 -> 2
Other:
- board text added: "Designed by Philip McGaw https://philipmcgaw.com"
