File: Woggle/Woggle.kicad_sch (KiCad schematic)
At the start: 21 parts, among them J1 ICSP, SW1 SW_SPDT, SW2 SW_Push, U1 ATtiny85-20P

Commit message: .
Parts:
- added Lanyard1: MountingHole, MountingHole:MountingHole_5mm, symbol Mechanical:MountingHole
- renumbered D7 to D1, D6 to D10, D1 to D2, D8 to D4, D2 to D5, D4 to D6, D9 to D7, D10 to D8, D5 to D9
Changed lines of the file:
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@@
 		(dnp no)
 		(fields_autoplaced yes)
-		(property "Reference" "D5"
+		(property "Reference" "D9"
 			(at 236.22 101.5364 90)
 			(effects
@@
 			(project "Woggle"
 				(path "/babca5d2-1380-4e56-a1f5-28dbd0ec42c7"
-					(reference "D5")
+					(reference "D9")
 					(unit 1)
 				)
@@
 		(dnp no)
 		(fields_autoplaced yes)
-		(property "Reference" "#PWR04"
+		(property "Reference" "#PWR02"
 			(at 57.15 74.93 0)
 			(effects
@@
 			(project ""
 				(path "/babca5d2-1380-4e56-a1f5-28dbd0ec42c7"
-					(reference "#PWR04")
+					(reference "#PWR02")
+					(unit 1)
+				)
+			)
+		)
+	)
+	(symbol
+		(lib_id "Mechanical:MountingHole")
+		(at 257.81 27.94 0)
+		(unit 1)
+		(exclude_from_sim no)
+		(in_bom no)
+		(on_board yes)
+		(dnp no)
+		(fields_autoplaced yes)
+		(property "Reference" "Lanyard1"
+			(at 260.35 26.6699 0)
+			(effects
+				(font
+					(size 1.27 1.27)
+				)
+				(justify left)
+			)
+		)
+		(property "Value" "MountingHole"
+			(at 260.35 29.2099 0)
+			(effects
+				(font
+					(size 1.27 1.27)
+				)
+				(justify left)
+			)
+		)
+		(property "Footprint" "MountingHole:MountingHole_5mm"
+			(at 257.81 27.94 0)
+			(effects
+				(font
+					(size 1.27 1.27)
+				)
+				(hide yes)
+			)
+		)
+		(property "Datasheet" "~"
+			(at 257.81 27.94 0)
+			(effects
+				(font
+					(size 1.27 1.27)
+				)
+				(hide yes)
+			)
+		)
+		(property "Description" "Mounting Hole without connection"
+			(at 257.81 27.94 0)
+			(effects
+				(font
+					(size 1.27 1.27)
+				)
+				(hide yes)
+			)
+		)
+		(instances
+			(project ""
+				(path "/babca5d2-1380-4e56-a1f5-28dbd0ec42c7"
+					(reference "Lanyard1")
 					(unit 1)
 				)
@@
 		(dnp no)
 		(fields_autoplaced yes)
-		(property "Reference" "#PWR06"
+		(property "Reference" "#PWR05"
 			(at 142.24 68.58 0)
 			(effects
@@
 			(project "Woggle"
 				(path "/babca5d2-1380-4e56-a1f5-28dbd0ec42c7"
-					(reference "#PWR06")
+					(reference "#PWR05")
 					(unit 1)
 				)
@@
 		(dnp no)
 		(fields_autoplaced yes)
-		(property "Reference" "D4"
+		(property "Reference" "D6"
 			(at 218.44 101.6634 90)
 			(effects
@@
 			(project "Woggle"
 				(path "/babca5d2-1380-4e56-a1f5-28dbd0ec42c7"
-					(reference "D4")
+					(reference "D6")
 					(unit 1)
 				)
@@
 		(dnp no)
 		(fields_autoplaced yes)
-		(property "Reference" "D7"
+		(property "Reference" "D1"
 			(at 209.55 81.2164 90)
 			(effects
@@
 			(project "Woggle"
 				(path "/babca5d2-1380-4e56-a1f5-28dbd0ec42c7"
-					(reference "D7")
+					(reference "D1")
 					(unit 1)
 				)
@@
 		(dnp no)
 		(fields_autoplaced yes)
-		(property "Reference" "#PWR03"
+		(property "Reference" "#PWR06"
 			(at 142.24 106.68 0)
 			(effects
@@
 			(project "Woggle"
 				(path "/babca5d2-1380-4e56-a1f5-28dbd0ec42c7"
-					(reference "#PWR03")
+					(reference "#PWR06")
 					(unit 1)
 				)
@@
 		(dnp no)
 		(fields_autoplaced yes)
-		(property "Reference" "D9"
+		(property "Reference" "D7"
 			(at 226.06 81.2164 90)
 			(effects
@@
 			(project "Woggle"
 				(path "/babca5d2-1380-4e56-a1f5-28dbd0ec42c7"
-					(reference "D9")
+					(reference "D7")
 					(unit 1)
 				)
@@
 		(dnp no)
 		(fields_autoplaced yes)
-		(property "Reference" "D1"
+		(property "Reference" "D2"
 			(at 209.55 91.3764 90)
 			(effects
@@
 			(project ""
 				(path "/babca5d2-1380-4e56-a1f5-28dbd0ec42c7"
-					(reference "D1")
+					(reference "D2")
 					(unit 1)
 				)
@@
 		(dnp no)
 		(fields_autoplaced yes)
-		(property "Reference" "D2"
+		(property "Reference" "D5"
 			(at 218.44 91.5034 90)
 			(effects
@@
 			(project "Woggle"
 				(path "/babca5d2-1380-4e56-a1f5-28dbd0ec42c7"
-					(reference "D2")
+					(reference "D5")
 					(unit 1)
 				)
@@
 		(dnp no)
 		(fields_autoplaced yes)
-		(property "Reference" "D8"
+		(property "Reference" "D4"
 			(at 218.44 81.3434 90)
 			(effects
@@
 			(project "Woggle"
 				(path "/babca5d2-1380-4e56-a1f5-28dbd0ec42c7"
-					(reference "D8")
+					(reference "D4")
 					(unit 1)
 				)
@@
 		(dnp no)
 		(fields_autoplaced yes)
-		(property "Reference" "#PWR05"
+		(property "Reference" "#PWR03"
 			(at 102.87 80.01 0)
 			(effects
@@
 			(project "Woggle"
 				(path "/babca5d2-1380-4e56-a1f5-28dbd0ec42c7"
-					(reference "#PWR05")
+					(reference "#PWR03")
 					(unit 1)
 				)
@@
 		(dnp no)
 		(fields_autoplaced yes)
-		(property "Reference" "D6"
+		(property "Reference" "D10"
 			(at 245.11 101.6634 90)
 			(effects
@@
 			(project "Woggle"
 				(path "/babca5d2-1380-4e56-a1f5-28dbd0ec42c7"
-					(reference "D6")
+					(reference "D10")
 					(unit 1)
 				)
@@
 		(dnp no)
 		(fields_autoplaced yes)
-		(property "Reference" "D10"
+		(property "Reference" "D8"
 			(at 234.95 81.3434 90)
 			(effects
@@
 			(project "Woggle"
 				(path "/babca5d2-1380-4e56-a1f5-28dbd0ec42c7"
-					(reference "D10")
+					(reference "D8")
 					(unit 1)
 				)
@@
 		(dnp no)
 		(fields_autoplaced yes)
-		(property "Reference" "#PWR02"
+		(property "Reference" "#PWR04"
 			(at 102.87 92.71 0)
 			(effects
@@
 			(project "Woggle"
 				(path "/babca5d2-1380-4e56-a1f5-28dbd0ec42c7"
-					(reference "#PWR02")
-					(unit 1)
-				)
+					(reference "#PWR04")
+					(unit 1)
+				)

Commit message: .
Parts:
- J1: footprint Connector_PinHeader_2.54mm:PinHeader_2x03_P2.54mm_Vertical -> Connector:Tag-Connect_TC2030-IDC-NL_2x03_P1.27mm_Vertical
- R1, R2, R3, R4: value R_Small -> 390
- SW1: footprint (none) -> Button_Switch_THT:SW_Slide_SPDT_Angled_CK_OS102011MA1Q
- SW2: footprint (none) -> Button_Switch_THT:SW_PUSH-12mm
Connections:
- net MISO/ARD12: now also R1.1; no longer R2.1
- net SCK/ARD13: now also R2.1; no longer R1.1
Other:
- note added: "Assume that we will want to current limit each LED to about 5 mA, these values will need to be adjusted due to duty cycle to ensure they are bright enouth https://philipmcgaw.com/led-resistors/"
- moved on the sheet: BT1, J1, Lanyard1, SW1

Commit message: .
Parts:
- added C1: 0.1uf, Franzininho:C025-025X050, symbol Device:C_Small
- added C2: 10uF, Capacitors_THT:CP_Radial_D5.0mm_P2.50mm, symbol Device:C_Polarized_Small
- added D13: Blink, LED_THT:LED_D5.0mm, symbol Device:LED_Small_Filled
- added D14: Power, LED_THT:LED_D5.0mm, symbol Device:LED_Small_Filled
- added D15, D17: BZT52, Diode_THT:D_5W_P10.16mm_Horizontal, symbol Device:D_Zener_Small_Filled
- added D16: 1N4148, Diode_THT:D_5W_P10.16mm_Horizontal, symbol Device:D_Small_Filled
- added R5, R9: 1K, Resistor_THT:R_Axial_DIN0207_L6.3mm_D2.5mm_P10.16mm_Horizontal, symbol Device:R_Small
- added R6: 1K5, Resistor_THT:R_Axial_DIN0207_L6.3mm_D2.5mm_P10.16mm_Horizontal, symbol Device:R_Small
- added R7, R8: 68R, Resistor_THT:R_Axial_DIN0207_L6.3mm_D2.5mm_P10.16mm_Horizontal, symbol Device:R_Small
- added SW3: Reset, Button_Switch_THT:SW_PUSH-12mm, symbol Switch:SW_Push
- added X1: USB-A-H, Connector_USB:USB_B_Lumberg_2411_02_Horizontal, symbol Connector:USB_B
- R1, R2, R3, R4: footprint Resistor_THT:R_Axial_DIN0204_L3.6mm_D1.6mm_P5.08mm_Horizontal -> Resistor_THT:R_Axial_DIN0207_L6.3mm_D2.5mm_P10.16mm_Horizontal
- SW2: value SW_Push -> Sequance
Connections:
- net GND: now also C1.2, C2.2, D15.2 (A), D17.2 (A), R5.1, R9.1, SW3.1, X1.4 (GND), X1.5 (Shield)
- net Reset/ARD10: now also SW3.2
- net at D1.2 (A), D11.2 (A), D12.1 (K)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: now also D13.2 (A)
- net at R3.1, U1.2 (XTAL1/PB3): now also R7.2
- net at R4.1, U1.3 (XTAL2/PB4): now also R8.2
- new net: D13.1 (K), R9.2
- new net: D16.2 (A), X1.1 (VBUS)
- new net: D14.1 (K), R5.2
- new net +5V: C1.1, C2.1, D14.2 (A), D16.1 (K), R6.1
- new net D+: D17.1 (K), R8.1, X1.3 (D+)
- new net D-: D15.1 (K), R6.2, R7.1, X1.2 (D-)
Other:
- moved on the sheet: BT1, D1, D10, D11, D12, D2, D3, D4, D5, D6, D7, D8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

Commit message: .
Parts:
- removed X1: USB-A-H, Connector_USB:USB_B_Lumberg_2411_02_Horizontal, symbol Connector:USB_B
- added J2: USB_Program, Connector_PinHeader_2.54mm:PinHeader_1x04_P2.54mm_Vertical, symbol Connector:Conn_01x04_Pin
- Lanyard1: value MountingHole -> Lanyard
Connections:
- net D+: now also J2.2 (Pin_2)
- net D-: now also J2.3 (Pin_3)
- net GND: now also J2.4 (Pin_4)
- net at D16.2 (A): now also J2.1 (Pin_1)
Changed lines of the file:
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@@
-	)
-	(junction
-		(at 50.8 80.01)
-		(diameter 0)
-		(color 0 0 0 0)
 	)
 	(junction
@@
 	(wire
 		(pts
-			(xy 50.8 80.01) (xy 50.8 82.55)
+			(xy 58.42 72.39) (xy 58.42 78.74)
 		)
 		(stroke
@@
 	(wire
 		(pts
-			(xy 48.26 80.01) (xy 50.8 80.01)
-		)
-		(stroke
-			(width 0)
-			(type default)
-		)
-	)
-	(wire
-		(pts
 			(xy 63.5 90.17) (xy 63.5 95.25)
 		)
@@
 	(wire
 		(pts
-			(xy 48.26 77.47) (xy 48.26 80.01)
-		)
-		(stroke
-			(width 0)
-			(type default)
-		)
-	)
-	(wire
-		(pts
 			(xy 179.07 54.61) (xy 193.04 54.61)
 		)
@@
 	(wire
 		(pts
-			(xy 58.42 62.23) (xy 68.58 62.23)
+			(xy 58.42 64.77) (xy 68.58 64.77)
 		)
 		(stroke
@@
 	(wire
 		(pts
-			(xy 50.8 77.47) (xy 50.8 80.01)
-		)
-		(stroke
-			(width 0)
-			(type default)
-		)
-	)
-	(wire
-		(pts
 			(xy 234.95 54.61) (xy 234.95 67.31)
 		)
@@
 	(wire
 		(pts
-			(xy 68.58 57.15) (xy 68.58 62.23)
+			(xy 68.58 57.15) (xy 68.58 64.77)
 		)
 		(stroke
@@
 	)
 	(symbol
-		(lib_id "Connector:USB_B")
-		(at 50.8 67.31 0)
-		(unit 1)
-		(exclude_from_sim no)
-		(in_bom yes)
-		(on_board yes)
-		(dnp no)
-		(fields_autoplaced yes)
-		(property "Reference" "X1"
-			(at 50.8 54.61 0)
-			(effects
-				(font
-					(size 1.4986 1.4986)
-				)
-			)
-		)
-		(property "Value" "USB-A-H"
-			(at 50.8 57.15 0)
-			(effects
-				(font
-					(size 1.4986 1.4986)
-				)
-			)
-		)
-		(property "Footprint" "Connector_USB:USB_B_Lumberg_2411_02_Horizontal"
-			(at 54.61 68.58 0)
-			(effects
-				(font
-					(size 1.27 1.27)
-				)
-				(hide yes)
-			)
-		)
-		(property "Datasheet" "~"
-			(at 54.61 68.58 0)
-			(effects
-				(font
-					(size 1.27 1.27)
-				)
-				(hide yes)
-			)
-		)
-		(property "Description" "USB Type B connector"
-			(at 50.8 67.31 0)
-			(effects
-				(font
-					(size 1.27 1.27)
-				)
-				(hide yes)
-			)
-		)
-		(pin "2"
-		)
-		(pin "5"
-		)
-		(pin "4"
-		)
-		(pin "1"
-		)
-		(pin "3"
-		)
-		(instances
-			(project "Woggle"
-				(path "/babca5d2-1380-4e56-a1f5-28dbd0ec42c7"
-					(reference "X1")
-					(unit 1)
-				)
-			)
-		)
-	)
-	(symbol
 		(lib_id "Device:R_Small")
 		(at 251.46 54.61 270)
@@
 	(symbol
 		(lib_id "power:GND")
-		(at 50.8 82.55 0)
+		(at 58.42 78.74 0)
 		(unit 1)
 		(exclude_from_sim no)
@@
 		(fields_autoplaced yes)
 		(property "Reference" "#PWR016"
-			(at 50.8 88.9 0)
+			(at 58.42 85.09 0)
 			(effects
 				(font
@@
 		)
 		(property "Value" "GND"
-			(at 53.34 83.8199 0)
-			(effects
-				(font
-					(size 1.27 1.27)
-				)
-				(justify left)
+			(at 58.42 83.82 0)
+			(effects
+				(font
+					(size 1.27 1.27)
+				)
 			)
 		)
 		(property "Footprint" ""
-			(at 50.8 82.55 0)
+			(at 58.42 78.74 0)
 			(effects
 				(font
@@
 		)
 		(property "Datasheet" ""
-			(at 50.8 82.55 0)
+			(at 58.42 78.74 0)
 			(effects
 				(font
@@
 		)
 		(property "Description" "Power symbol creates a global label with name \"GND\" , ground"
-			(at 50.8 82.55 0)
+			(at 58.42 78.74 0)
 			(effects
 				(font
@@
 				(path "/babca5d2-1380-4e56-a1f5-28dbd0ec42c7"
 					(reference "#PWR016")
+					(unit 1)
+				)
+			)
+		)
+	)
+	(symbol
+		(lib_id "Connector:Conn_01x04_Pin")
+		(at 53.34 67.31 0)
+		(unit 1)
+		(exclude_from_sim no)
+		(in_bom yes)
+		(on_board yes)
+		(dnp no)
+		(fields_autoplaced yes)
+		(property "Reference" "J2"
+			(at 53.975 59.69 0)
+			(effects
+				(font
+					(size 1.27 1.27)
+				)
+			)
+		)
+		(property "Value" "USB_Program"
+			(at 53.975 62.23 0)
+			(effects
+				(font
+					(size 1.27 1.27)
+				)
+			)
+		)
+		(property "Footprint" "Connector_PinHeader_2.54mm:PinHeader_1x04_P2.54mm_Vertical"
+			(at 53.34 67.31 0)
+			(effects
+				(font
+					(size 1.27 1.27)
+				)
+				(hide yes)
+			)
+		)
+		(property "Datasheet" "~"
+			(at 53.34 67.31 0)
+			(effects
+				(font
+					(size 1.27 1.27)
+				)
+				(hide yes)
+			)
+		)
+		(property "Description" "Generic connector, single row, 01x04, script generated"
+			(at 53.34 67.31 0)
+			(effects
+				(font
+					(size 1.27 1.27)
+				)
+				(hide yes)
+			)
+		)
+		(pin "3"
+		)
+		(pin "2"
+		)
+		(pin "4"
+		)
+		(pin "1"
+		)
+		(instances
+			(project ""
+				(path "/babca5d2-1380-4e56-a1f5-28dbd0ec42c7"
+					(reference "J2")
 					(unit 1)
 				)
@@
 			)
 		)
-		(property "Value" "MountingHole"
+		(property "Value" "Lanyard"
 			(at 160.02 120.6499 0)
 			(effects

Commit message: .
Parts:
- removed D13: Blink, LED_THT:LED_D5.0mm, symbol Device:LED_Small_Filled
- removed D14: Power, LED_THT:LED_D5.0mm, symbol Device:LED_Small_Filled
- removed D15, D17: BZT52, Diode_THT:D_5W_P10.16mm_Horizontal, symbol Device:D_Zener_Small_Filled
- removed D16: 1N4148, Diode_THT:D_5W_P10.16mm_Horizontal, symbol Device:D_Small_Filled
- removed J1: ICSP, Connector:Tag-Connect_TC2030-IDC-NL_2x03_P1.27mm_Vertical, symbol Connector_Generic:Conn_02x03_Odd_Even
- removed J2: USB_Program, Connector_PinHeader_2.54mm:PinHeader_1x04_P2.54mm_Vertical, symbol Connector:Conn_01x04_Pin
- removed R5, R9: 1K, Resistor_THT:R_Axial_DIN0207_L6.3mm_D2.5mm_P10.16mm_Horizontal, symbol Device:R_Small
- removed R6: 1K5, Resistor_THT:R_Axial_DIN0207_L6.3mm_D2.5mm_P10.16mm_Horizontal, symbol Device:R_Small
- removed R7, R8: 68R, Resistor_THT:R_Axial_DIN0207_L6.3mm_D2.5mm_P10.16mm_Horizontal, symbol Device:R_Small
- removed SW3: Reset, Button_Switch_THT:SW_PUSH-12mm, symbol Switch:SW_Push
- BT1: footprint (none) -> Scouts:2 x AAA battery cell holder
- D1, D10, D11, D12, D2, D3, D4, D5, D6, D7, D8, D9: footprint LED_THT:LED_D5.0mm -> Scouts:5mm LED
- U1: footprint Package_DIP:DIP-8_W7.62mm -> Scouts:DIP 8
Connections:
- net MISO/ARD12: no longer names the net of R1.1, U1.6 (PB1)
- net MOSI/ARD11: no longer names the net of SW2.1, U1.5 (AREF/PB0)
- net Reset/ARD10: no longer names the net of U1.1 (~{RESET}/PB5)
- net SCK/ARD13: no longer names the net of R2.1, U1.7 (PB2)
Other:
- moved on the sheet: BT1, C1, C2, Lanyard1, SW1

Commit message: .
Parts:
- D1: value 1a -> 1
- D10: value 5b -> 7
- D11: value 6a -> 2
- D12: value 6b -> 3
- D2: value 2a -> 10
- D3: value 3a -> 5
- D4: value 1b -> 0
- D5: value 2b -> 11
- D6: value 3b -> 4
- D7: value 4a -> 8
- D8: value 4b -> 9
- D9: value 5a -> 6
Connections:
- net at D10.2 (A), D11.1 (K), D12.2 (A)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: now also R4.1; no longer R4.2
- net at D2.1 (K), D3.2 (A), D5.2 (A)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: now also R3.1; no longer R3.2
- net at U1.2 (XTAL1/PB3): now also R3.2; no longer R3.1
- net at U1.3 (XTAL2/PB4): now also R4.2; no longer R4.1
Other:
- moved on the sheet: BT1, C1, C2, D1, D10, D11, D12, D2, D3, D4, D5, D6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

Commit message: .
Parts:
- removed C2: 10uF, Capacitors_THT:CP_Radial_D5.0mm_P2.50mm, symbol Device:C_Polarized_Small
- added C2: 100nF, Capacitor_THT:C_Disc_D4.7mm_W2.5mm_P5.00mm, symbol Device:C_Small
- C1: value 0.1uf -> 10pF; footprint Franzininho:C025-025X050 -> Capacitor_THT:C_Disc_D4.7mm_W2.5mm_P5.00mm; code (none) -> 100
- D1: value 1 -> LED 1
- D10: value 7 -> LED 7
- D11: value 2 -> LED 2
- D12: value 3 -> LED 3
- D2: value 10 -> LED 10
- D3: value 5 -> LED 5
- D4: value 0 -> LED 0
- D5: value 11 -> LED 11
- D6: value 4 -> LED 4
- D7: value 8 -> LED 8
- D8: value 9 -> LED 9
- D9: value 6 -> LED 6
Connections:
- net +5V is gone; now on net +VE: C1.1
- net +VE: now also C2.1
- net GND: now also C2.2
Other:
- moved on the sheet: D1, D10, D11, D12, D2, D3, D4, D5, D6, D7, D8, D9

Commit message: .
Parts:
- BT1: footprint Scouts:2 x AAA battery cell holder -> Scouts:Scouts - 2 x AAA battery cell holder
- D1, D10, D11, D12, D2, D3, D4, D5, D6, D7, D8, D9: footprint Scouts:5mm LED -> Scouts:Scouts - 5mm LED
- R1, R2, R3, R4: footprint Resistor_THT:R_Axial_DIN0207_L6.3mm_D2.5mm_P10.16mm_Horizontal -> Scouts:Scouts - Resistor (10.16mm)
- U1: footprint Scouts:DIP 8 -> Scouts:Scouts - DIP 8
